Commit message: com3

File: mp_bot_description/urdf/ros2_control.xacro (robot description, xacro)
@@ -62,208 +62,208 @@
       </joint>
     </ros2_control>
+    <ros2_control name="fr_arm" type="system">
+    <hardware>
+      <plugin>gazebo_ros2_control/GazeboSystem</plugin>
+    </hardware>
+    <joint name="fr_coxa_to_baselink">
+      <command_interface name="position">
+        <param name="min">1.658063</param>
+        <param name="max">-0.523599</param>
+      </command_interface>
+      <command_interface name="velocity">
+        <param name="min">-3.15</param>
+        <param name="max">3.15</param>
+      </command_interface>
+      <state_interface name="position">
+        <xacro:coxa_initial></xacro:coxa_initial>
+      </state_interface>
+      <state_interface name="velocity"/>
+      <state_interface name="effort"/>
+    </joint>
+    <joint name="fr_femur_to_coxa">
+      <command_interface name="position">
+        <param name="min">0.087266</param>
+        <param name="max">-2.70526</param>
+      </command_interface>
+      <command_interface name="velocity">
+        <param name="min">-3.15</param>
+        <param name="max">3.15</param>
+      </command_interface>
+      <state_interface name="position">
+        <xacro:femur_initial></xacro:femur_initial>
+      </state_interface>
+      <state_interface name="velocity"/>
+      <state_interface name="effort"/>
+    </joint>
+    <joint name="fr_tibia_to_femur">
+      <command_interface name="position">
+        <param name="min">0.087266</param>
+        <param name="max">-2.70526</param>
+      </command_interface>
+      <command_interface name="velocity">
+        <param name="min">-3.15</param>
+        <param name="max">3.15</param>
+      </command_interface>
+      <state_interface name="position">
+        <xacro:tibia_initial></xacro:tibia_initial>
+      </state_interface>
+      <state_interface name="velocity"/>
+      <state_interface name="effort"/>
+    </joint>
+  </ros2_control>
+  <ros2_control name="fl_arm" type="system">
+    <hardware>
+      <plugin>gazebo_ros2_control/GazeboSystem</plugin>
+    </hardware>
+    <joint name="fl_coxa_to_baselink">
+      <command_interface name="position">
+        <param name="min">1.658063</param>
+        <param name="max">-0.523599</param>
+      </command_interface>
+      <command_interface name="velocity">
+        <param name="min">-3.15</param>
+        <param name="max">3.15</param>
+      </command_interface>
+      <state_interface name="position">
+        <xacro:coxa_initial></xacro:coxa_initial>
+      </state_interface>
+      <state_interface name="velocity"/>
+      <state_interface name="effort"/>
+    </joint>
+    <joint name="fl_femur_to_coxa">
+      <command_interface name="position">
+        <param name="min">0.087266</param>
+        <param name="max">-2.70526</param>
+      </command_interface>
+      <command_interface name="velocity">
+        <param name="min">-3.15</param>
+        <param name="max">3.15</param>
+      </command_interface>
+      <state_interface name="position">
+        <xacro:femur_initial></xacro:femur_initial>
+      </state_interface>
+      <state_interface name="velocity"/>
+      <state_interface name="effort"/>
+    </joint>
+    <joint name="fl_tibia_to_femur">
+      <command_interface name="position">
+        <param name="min">0.087266</param>
+        <param name="max">-2.70526</param>
+      </command_interface>
+      <command_interface name="velocity">
+        <param name="min">-3.15</param>
+        <param name="max">3.15</param>
+      </command_interface>
+      <state_interface name="position">
+        <xacro:tibia_initial></xacro:tibia_initial>
+      </state_interface>
+      <state_interface name="velocity"/>
+      <state_interface name="effort"/>
+    </joint>
+  </ros2_control>
+  <ros2_control name="rr_arm" type="system">
+    <hardware>
+      <plugin>gazebo_ros2_control/GazeboSystem</plugin>
+    </hardware>
+    <joint name="rr_coxa_to_baselink">
+      <command_interface name="position">
+        <param name="min">1.658063</param>
+        <param name="max">-0.523599</param>
+      </command_interface>
+      <command_interface name="velocity">
+        <param name="min">-3.15</param>
+        <param name="max">3.15</param>
+      </command_interface>
+      <state_interface name="position">
+        <xacro:coxa_initial></xacro:coxa_initial>
+      </state_interface>
+      <state_interface name="velocity"/>
+      <state_interface name="effort"/>
+    </joint>
+    <joint name="rr_femur_to_coxa">
+      <command_interface name="position">
+        <param name="min">0.087266</param>
+        <param name="max">-2.70526</param>
+      </command_interface>
+      <command_interface name="velocity">
+        <param name="min">-3.15</param>
+        <param name="max">3.15</param>
+      </command_interface>
+      <state_interface name="position">
+        <xacro:femur_initial></xacro:femur_initial>
+      </state_interface>
+      <state_interface name="velocity"/>
+      <state_interface name="effort"/>
+    </joint>
+    <joint name="rr_tibia_to_femur">
+      <command_interface name="position">
+        <param name="min">0.087266</param>
+        <param name="max">-2.70526</param>
+      </command_interface>
+      <command_interface name="velocity">
+        <param name="min">-3.15</param>
+        <param name="max">3.15</param>
+      </command_interface>
+      <state_interface name="position">
+        <xacro:tibia_initial></xacro:tibia_initial>
+      </state_interface>
+      <state_interface name="velocity"/>
+      <state_interface name="effort"/>
+    </joint>
+  </ros2_control>
+  <ros2_control name="rl_arm" type="system">
+    <hardware>
+      <plugin>gazebo_ros2_control/GazeboSystem</plugin>
+    </hardware>
+    <joint name="rl_coxa_to_baselink">
+      <command_interface name="position">
+        <param name="min">1.658063</param>
+        <param name="max">-0.523599</param>
+      </command_interface>
+      <command_interface name="velocity">
+        <param name="min">-3.15</param>
+        <param name="max">3.15</param>
+      </command_interface>
+      <state_interface name="position">
+        <xacro:coxa_initial></xacro:coxa_initial>
+      </state_interface>
+      <state_interface name="velocity"/>
+      <state_interface name="effort"/>
+    </joint>
+    <joint name="rl_femur_to_coxa">
+      <command_interface name="position">
+        <param name="min">0.087266</param>
+        <param name="max">-2.70526</param>
+      </command_interface>
+      <command_interface name="velocity">
+        <param name="min">-3.15</param>
+        <param name="max">3.15</param>
+      </command_interface>
+      <state_interface name="position">
+        <xacro:femur_initial></xacro:femur_initial>
+      </state_interface>
+      <state_interface name="velocity"/>
+      <state_interface name="effort"/>
+    </joint>
+    <joint name="rl_tibia_to_femur">
+      <command_interface name="position">
+        <param name="min">0.087266</param>
+        <param name="max">-2.70526</param>
+      </command_interface>
+      <command_interface name="velocity">
+        <param name="min">-3.15</param>
+        <param name="max">3.15</param>
+      </command_interface>
+      <state_interface name="position">
+        <xacro:tibia_initial></xacro:tibia_initial>
+      </state_interface>
+      <state_interface name="velocity"/>
+      <state_interface name="effort"/>
+    </joint>
+  </ros2_control>
   </xacro:if>
-  <ros2_control name="fr_arm" type="system">
-    <hardware>
-      <plugin>gazebo_ros2_control/GazeboSystem</plugin>
-    </hardware>
-    <joint name="fr_coxa_to_baselink">
-      <command_interface name="position">
-        <param name="min">1.658063</param>
-        <param name="max">-0.523599</param>
-      </command_interface>
-      <command_interface name="velocity">
-        <param name="min">-3.15</param>
-        <param name="max">3.15</param>
-      </command_interface>
-      <state_interface name="position">
-        <xacro:coxa_initial></xacro:coxa_initial>
-      </state_interface>
-      <state_interface name="velocity"/>
-      <state_interface name="effort"/>
-    </joint>
-    <joint name="fr_femur_to_coxa">
-      <command_interface name="position">
-        <param name="min">0.087266</param>
-        <param name="max">-2.70526</param>
-      </command_interface>
-      <command_interface name="velocity">
-        <param name="min">-3.15</param>
-        <param name="max">3.15</param>
-      </command_interface>
-      <state_interface name="position">
-        <xacro:femur_initial></xacro:femur_initial>
-      </state_interface>
-      <state_interface name="velocity"/>
-      <state_interface name="effort"/>
-    </joint>
-    <joint name="fr_tibia_to_femur">
-      <command_interface name="position">
-        <param name="min">0.087266</param>
-        <param name="max">-2.70526</param>
-      </command_interface>
-      <command_interface name="velocity">
-        <param name="min">-3.15</param>
-        <param name="max">3.15</param>
-      </command_interface>
-      <state_interface name="position">
-        <xacro:tibia_initial></xacro:tibia_initial>
-      </state_interface>
-      <state_interface name="velocity"/>
-      <state_interface name="effort"/>
-    </joint>
-  </ros2_control>
-  <ros2_control name="fl_arm" type="system">
-    <hardware>
-      <plugin>gazebo_ros2_control/GazeboSystem</plugin>
-    </hardware>
-    <joint name="fl_coxa_to_baselink">
-      <command_interface name="position">
-        <param name="min">1.658063</param>
-        <param name="max">-0.523599</param>
-      </command_interface>
-      <command_interface name="velocity">
-        <param name="min">-3.15</param>
-        <param name="max">3.15</param>
-      </command_interface>
-      <state_interface name="position">
-        <xacro:coxa_initial></xacro:coxa_initial>
-      </state_interface>
-      <state_interface name="velocity"/>
-      <state_interface name="effort"/>
-    </joint>
-    <joint name="fl_femur_to_coxa">
-      <command_interface name="position">
-        <param name="min">0.087266</param>
-        <param name="max">-2.70526</param>
-      </command_interface>
-      <command_interface name="velocity">
-        <param name="min">-3.15</param>
-        <param name="max">3.15</param>
-      </command_interface>
-      <state_interface name="position">
-        <xacro:femur_initial></xacro:femur_initial>
-      </state_interface>
-      <state_interface name="velocity"/>
-      <state_interface name="effort"/>
-    </joint>
-    <joint name="fl_tibia_to_femur">
-      <command_interface name="position">
-        <param name="min">0.087266</param>
-        <param name="max">-2.70526</param>
-      </command_interface>
-      <command_interface name="velocity">
-        <param name="min">-3.15</param>
-        <param name="max">3.15</param>
-      </command_interface>
-      <state_interface name="position">
-        <xacro:tibia_initial></xacro:tibia_initial>
-      </state_interface>
-      <state_interface name="velocity"/>
-      <state_interface name="effort"/>
-    </joint>
-  </ros2_control>
-  <ros2_control name="rr_arm" type="system">
-    <hardware>
-      <plugin>gazebo_ros2_control/GazeboSystem</plugin>
-    </hardware>
-    <joint name="rr_coxa_to_baselink">
-      <command_interface name="position">
-        <param name="min">1.658063</param>
-        <param name="max">-0.523599</param>
-      </command_interface>
-      <command_interface name="velocity">
-        <param name="min">-3.15</param>
-        <param name="max">3.15</param>
-      </command_interface>
-      <state_interface name="position">
-        <xacro:coxa_initial></xacro:coxa_initial>
-      </state_interface>
-      <state_interface name="velocity"/>
-      <state_interface name="effort"/>
-    </joint>
-    <joint name="rr_femur_to_coxa">
-      <command_interface name="position">
-        <param name="min">0.087266</param>
-        <param name="max">-2.70526</param>
-      </command_interface>
-      <command_interface name="velocity">
-        <param name="min">-3.15</param>
-        <param name="max">3.15</param>
-      </command_interface>
-      <state_interface name="position">
-        <xacro:femur_initial></xacro:femur_initial>
-      </state_interface>
-      <state_interface name="velocity"/>
-      <state_interface name="effort"/>
-    </joint>
-    <joint name="rr_tibia_to_femur">
-      <command_interface name="position">
-        <param name="min">0.087266</param>
-        <param name="max">-2.70526</param>
-      </command_interface>
-      <command_interface name="velocity">
-        <param name="min">-3.15</param>
-        <param name="max">3.15</param>
-      </command_interface>
-      <state_interface name="position">
-        <xacro:tibia_initial></xacro:tibia_initial>
-      </state_interface>
-      <state_interface name="velocity"/>
-      <state_interface name="effort"/>
-    </joint>
-  </ros2_control>
-  <ros2_control name="rl_arm" type="system">
-    <hardware>
-      <plugin>gazebo_ros2_control/GazeboSystem</plugin>
-    </hardware>
-    <joint name="rl_coxa_to_baselink">
-      <command_interface name="position">
-        <param name="min">1.658063</param>
-        <param name="max">-0.523599</param>
-      </command_interface>
-      <command_interface name="velocity">
-        <param name="min">-3.15</param>
-        <param name="max">3.15</param>
-      </command_interface>
-      <state_interface name="position">
-        <xacro:coxa_initial></xacro:coxa_initial>
-      </state_interface>
-      <state_interface name="velocity"/>
-      <state_interface name="effort"/>
-    </joint>
-    <joint name="rl_femur_to_coxa">
-      <command_interface name="position">
-        <param name="min">0.087266</param>
-        <param name="max">-2.70526</param>
-      </command_interface>
-      <command_interface name="velocity">
-        <param name="min">-3.15</param>
-        <param name="max">3.15</param>
-      </command_interface>
-      <state_interface name="position">
-        <xacro:femur_initial></xacro:femur_initial>
-      </state_interface>
-      <state_interface name="velocity"/>
-      <state_interface name="effort"/>
-    </joint>
-    <joint name="rl_tibia_to_femur">
-      <command_interface name="position">
-        <param name="min">0.087266</param>
-        <param name="max">-2.70526</param>
-      </command_interface>
-      <command_interface name="velocity">
-        <param name="min">-3.15</param>
-        <param name="max">3.15</param>
-      </command_interface>
-      <state_interface name="position">
-        <xacro:tibia_initial></xacro:tibia_initial>
-      </state_interface>
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